File: PCB/pcb.kicad_pcb (KiCad board)
At the start: 2 copper layers, 120 x 60 mm, 10 parts, among them J1 Conn_01x08_Pin, SW1 SW_Push, SW2 SW_Push, SW3 SW_Push, U1 XIAO-ESP32-C3-SMD

Commit message: Final Reviews
Parts:
- moved U1 66.2 mm to (141.4, 97.9), turned to 0 degrees
- moved SW3 64.9 mm to (98.1, 77.4)
- moved SW1 63.0 mm to (79.0, 77.4)
- moved SW2 50.6 mm to (117.0, 77.4)
- moved H1 26.1 mm to (147.5, 76.0)
- moved H2 26.0 mm to (147.5, 112.5)
- moved BZ1 25.0 mm to (129.7, 80.5)
- moved H4 7.52 mm to (61.0, 76.0)
- moved H3 7.02 mm to (61.0, 112.5)
Routing:
- net Net-(J1-Pin_6): track 25.2 -> 105.7 mm
- net Net-(J1-Pin_7): track 27.4 -> 98.5 mm
- net Net-(J1-Pin_5): track 37.6 -> 107.4 mm
- net Net-(J1-Pin_8): track 31.0 -> 87.9 mm
- net Net-(J1-Pin_2): track 26.8 -> 78.4 mm
- net Net-(J1-Pin_4): track 34.5 -> 82.7 mm
- net Net-(J1-Pin_3): track 31.4 -> 77.9 mm
- net GND: track 144.0 -> 113.2 mm
- net Net-(U1-D1): track 89.3 -> 112.7 mm
- net Net-(U1-D0): track 70.6 -> 84.5 mm
- net Net-(BZ1-+): track 23.0 -> 26.7 mm
Other:
- board size 120 x 60 mm -> 96.5 x 46 mm
